File: loopSwitchSTM.kicad_pcb (KiCad board)
At the start: 2 copper layers, 86 parts, among them J1 Conn_01x07_Socket, J10 SJ-63063B, J11 SJ-63063B, J12 SJ-63063B, J13 SJ-63063B, J14 SJ-63063B, J16 AudioJack4, J17 AudioJack4, J2 Jack-DC, J3 SJ-63063B, J4 SJ-63063B, J5 SJ-63063B, J6 SJ-63063B, J7 SJ-63063B, J8 SJ-63063B, J9 SJ-63063B, K1 G6S-2, K2 G6S-2, K3 G6S-2, K4 G6S-2, K5 G6S-2, Q1 IRLML2060, Q10 IRLML2060, Q11 IRLML2060, Q12 2N7002, Q13 2N7002, Q14 2N7002, Q2 2N7002, Q3 2N7002, Q4 2N7002, Q8 IRLML2060, Q9 IRLML2060, U1 74HC595, U2 H11L1

Commit message: PCB rev 0.1
Parts:
- moved FB1 9.94 mm to (111.5, 66.0)
- moved C16 8.74 mm to (137.2, 75.2)
- moved C2 8.74 mm to (115.2, 75.2)
- moved R26 8.74 mm to (128.5, 61.5)
- moved C15 8.74 mm to (131.0, 60.3)
- moved D6 8.74 mm to (138.0, 67.5)
- moved J11 8.74 mm to (162.8, 60.2)
- moved J17 8.74 mm to (125.9, 50.6)
- moved J2 8.74 mm to (113.2, 60.5)
- moved J4 8.74 mm to (208.5, 60.2)
- moved J7 8.74 mm to (193.3, 60.2)
- moved J9 8.74 mm to (178.1, 60.2)
- moved R27 8.74 mm to (125.9, 67.9)
- moved J13 8.74 mm to (147.6, 60.2)
- moved FB2 8.74 mm to (119.2, 66.9)
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Routing:
- net GND: track 0.00 -> 13.9 mm, vias 34 -> 36
- net GNDD: track 2.00 -> 9.12 mm
- net Net-(FB1-Pad1): track 14.1 -> 18.9 mm, vias 0 -> 1
- net unconnected-(R27-Pad1): track 8.50 -> 4.33 mm
- net +9V: track 112.6 -> 114.3 mm
- net Net-(FB1-Pad2): track 3.93 -> 5.39 mm
- net /1: track 101.9 -> 100.5 mm
- net Net-(Q1-G): track 1.94 -> 3.21 mm
- net +3.3V: track 33.8 -> 34.4 mm
