File: loopSwitchSTM.kicad_sch (KiCad schematic)
At the start: 86 parts, among them J1 Conn_01x07_Socket, J10 SJ-63063B, J11 SJ-63063B, J12 SJ-63063B, J13 SJ-63063B, J14 SJ-63063B, J16 AudioJack4, J17 AudioJack4, J2 Jack-DC, J3 SJ-63063B, J4 SJ-63063B, J5 SJ-63063B, J6 SJ-63063B, J7 SJ-63063B, J8 SJ-63063B, J9 SJ-63063B, K1 G6S-2, K2 G6S-2, K3 G6S-2, K4 G6S-2, K5 G6S-2, Q1 IRLML2060, Q10 IRLML2060, Q11 IRLML2060, Q12 2N7002, Q13 2N7002, Q14 2N7002, Q2 2N7002, Q3 2N7002, Q4 2N7002, Q8 IRLML2060, Q9 IRLML2060, U1 74HC595, U2 H11L1

Commit message: PCB rev 0.1
Parts:
- added R28: 470r, symbol Device:R
Connections:
- net +3.3V: now also R28.1
- net at U2.4: now also R28.2
Changed lines of the file:
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@@
 	)
 	(junction
+		(at 261.62 160.02)
+		(diameter 0)
+		(color 0 0 0 0)
+	)
+	(junction
 		(at 388.62 115.57)
 		(diameter 0)
@@
 	(wire
 		(pts
+			(xy 278.13 160.02) (xy 261.62 160.02)
+		)
+		(stroke
+			(width 0)
+			(type default)
+		)
+	)
+	(wire
+		(pts
 			(xy 381 78.74) (xy 381 88.9)
 		)
@@
 	(wire
 		(pts
+			(xy 254 167.64) (xy 278.13 167.64)
+		)
+		(stroke
+			(width 0)
+			(type default)
+		)
+	)
+	(wire
+		(pts
 			(xy 231.14 92.71) (xy 231.14 91.44)
 		)
@@
 	(wire
 		(pts
-			(xy 260.35 245.11) (xy 260.35 231.14)
+			(xy 260.35 245.11) (xy 260.35 229.87)
 		)
 		(stroke
@@
 	(wire
 		(pts
-			(xy 228.6 231.14) (xy 228.6 229.87)
-		)
-		(stroke
-			(width 0)
-			(type default)
-		)
-	)
-	(wire
-		(pts
 			(xy 80.01 45.72) (xy 80.01 55.88)
 		)
@@
 	(wire
 		(pts
-			(xy 260.35 231.14) (xy 228.6 231.14)
+			(xy 260.35 229.87) (xy 228.6 229.87)
 		)
 		(stroke
@@
 	(symbol
 		(lib_id "Device:R")
+		(at 278.13 163.83 0)
+		(unit 1)
+		(exclude_from_sim no)
+		(in_bom yes)
+		(on_board yes)
+		(dnp no)
+		(fields_autoplaced yes)
+		(property "Reference" "R28"
+			(at 280.67 162.5599 0)
+			(effects
+				(font
+					(size 1.27 1.27)
+				)
+				(justify left)
+			)
+		)
+		(property "Value" "470r"
+			(at 280.67 165.0999 0)
+			(effects
+				(font
+					(size 1.27 1.27)
+				)
+				(justify left)
+			)
+		)
+		(property "Footprint" ""
+			(at 276.352 163.83 90)
+			(effects
+				(font
+					(size 1.27 1.27)
+				)
+				(hide yes)
+			)
+		)
+		(property "Datasheet" "~"
+			(at 278.13 163.83 0)
+			(effects
+				(font
+					(size 1.27 1.27)
+				)
+				(hide yes)
+			)
+		)
+		(property "Description" "Resistor"
+			(at 278.13 163.83 0)
+			(effects
+				(font
+					(size 1.27 1.27)
+				)
+				(hide yes)
+			)
+		)
+		(pin "1"
+		)
+		(pin "2"
+		)
+		(instances
+			(project ""
+				(path "/2a6ab95e-cf9d-48e4-bf2a-ab3d54f2719c"
+					(reference "R28")
+					(unit 1)
+				)
+			)
+		)
+	)
+	(symbol
+		(lib_id "Device:R")
 		(at 264.16 105.41 0)
 		(unit 1)
@@
 		(on_board yes)
 		(dnp no)
-		(fields_autoplaced yes)
 		(property "Reference" "U1"
-			(at 230.7433 227.33 0)
+			(at 231.902 226.06 0)
 			(effects
 				(font
@@
 		)
 		(property "Value" "74HC595"
-			(at 230.7433 229.87 0)
+			(at 231.394 228.346 0)
 			(effects
 				(font
